File: Elétrica/Schematic_monitor/_autosave-Schematic_monitor.kicad_sch (KiCad schematic)
At the start: 49 parts, among them J1 Conn_01x04, J2 USB_B_Micro, J3 Eletrode 1, J4 Eletrode 2, SW1 SW_Push, SW2 SW_SPDT, U1 STM32F446RET6TR, U2 LM1117S-3.3, U3 MLX90614ESF-ACC-000-TU, U4 MAX30100EFD+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

Commit message: Att
Parts:
- added J?: Conn_01x06, symbol Connector_Generic:Conn_01x06
Connections:
- net ADC1-0: no longer names the net of U1.14 (PA0)
Other:
- moved on the sheet: U1
