File: Elétrica/Schematic_monitor/Schematic_monitor.kicad_pcb (KiCad board)
At the start: 2 copper layers, 73.7 x 59 mm, 64 parts, among them J1 Conn_01x04, J2 USB_B_Micro, J3 Eletrode 1, J4 Eletrode 2, J5 Conn_01x09, SW1 SW_Push, SW2 SW_SPDT, U1 STM32F446RET6TR, U2 LM1117S-3.3, U3 MLX90614ESF-ACC-000-TU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

Commit message: Multiparameter Monitor PCB
Routing:
- net +3.3VA: track 60.9 -> 63.9 mm

Commit message: PRJ4
Routing:
- net VBUS: track 143.1 -> 142.5 mm
- net +3.3V: track 118.9 -> 118.3 mm
- removed copper zone on B.Cu, net GND
- removed copper zone on F.Cu, net GND

Commit message: prj4 - final
Parts:
- moved U2 46.2 mm to (109.4, 96.5), turned to 180 degrees
- moved C1 29.9 mm to (121.7, 99.6), turned to -90 degrees
- moved C2 28.2 mm to (121.7, 91.9), turned to 90 degrees
- moved FB2 22.8 mm to (124.7, 98.2), turned to -90 degrees
- moved FB1 21.2 mm to (124.7, 94.1), turned to 90 degrees
- moved U4 10.3 mm to (149.9, 97.1), turned to 0 degrees
- moved R11 9.17 mm to (147.1, 94.8), turned to -90 degrees
- moved R12 6.06 mm to (147.1, 98.1), turned to -90 degrees
Routing:
- net +3.3VA: track 63.9 -> 35.8 mm
- net VBUS: track 142.5 -> 154.9 mm, vias 4 -> 3
- net oxi_scl: track 24.9 -> 32.5 mm
- net Net-(U2-VO): track 24.9 -> 20.3 mm
- net +3.3V: track 118.3 -> 122.3 mm
- net oxi_sda: track 26.1 -> 28.7 mm
- net displ_sck: track 37.7 -> 36.8 mm
- added copper zone on B.Cu, net GND
- added copper zone on F.Cu, net GND
