File: Elétrica/Schematic_monitor/Schematic_monitor.kicad_pcb (KiCad board)
At the start: 2 copper layers, 64.1 x 51.3 mm, 62 parts, among them J1 Conn_01x04, J2 USB_B_Micro, J3 Eletrode 1, J4 Eletrode 2, J5 Conn_01x09, SW1 SW_Push, SW2 SW_SPDT, U1 STM32F446RET6TR, U2 LM1117S-3.3, U3 MLX90614ESF-ACC-000-TU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

Commit message: PRJ4 - Entregue
Parts:
- moved SW1 0.17 mm to (153.9, 129.8)
Routing:
- net VBUS: track 155.1 -> 164.3 mm
- net Net-(U2-VO): track 20.3 -> 27.6 mm
- net +3.3V: track 122.6 -> 127.4 mm
- net +3.3VA: track 35.8 -> 38.4 mm
- net Vref: track 27.4 -> 29.5 mm
- net GND: track 2.69 -> 0.93 mm, vias 8 -> 7
- net displ_led: track 44.5 -> 45.7 mm
- net Net-(U7A-+): track 13.2 -> 14.1 mm
- net displ_rst: track 52.6 -> 53.6 mm
- net Temp_SDA: track 23.8 -> 24.6 mm
- net HSE_IN: track 8.24 -> 9.02 mm
- net ADC1-1: track 25.9 -> 25.2 mm
- net oxi_scl: track 32.5 -> 33.1 mm
- net Net-(U6A-+): track 5.76 -> 5.55 mm, vias 1 -> 0
- net /sw_boot: track 8.95 -> 8.93 mm, vias 1 -> 0
Other:
- board text added: "Monitor Multiparâmetros V1.0"
- board text removed: "Monitor Multiparâmetros V0.7"

Commit message: Mudanças PRJ5 e PRJ4
Parts:
- added D5: LED, LED_SMD:LED_1210_3225Metric, F.Cu at (139.6, 116.6)
- added R16: 1k, Resistor_SMD:R_0805_2012Metric_Pad1.20x1.40mm_HandSolder, F.Cu at (133.1, 119.3)
- moved C10 44.5 mm to (138.7, 112.3)
- moved C8 44.5 mm to (124.9, 102.1)
- moved R1 44.5 mm to (141.9, 103.6)
- moved R3 44.5 mm to (110.3, 119.9)
- moved C15 44.5 mm to (119.0, 113.0)
- moved C18 44.5 mm to (123.3, 119.3)
- moved C3 44.5 mm to (127.8, 95.7)
- moved D3 44.5 mm to (115.8, 103.0)
- moved G*** 44.5 mm to (122.2, 126.8)
- moved J5 44.5 mm to (93.9, 107.3)
- moved R2 44.5 mm to (110.4, 116.2)
- moved R9 44.5 mm to (112.2, 103.4)
- moved U7 44.5 mm to (105.3, 111.8)
- moved C6 44.5 mm to (140.8, 99.3)
- moved J4 44.5 mm to (114.0, 127.4)
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Connections:
- U1 pad 42: unconnected-(U1-PA9-Pad42) -> led_pin
Routing:
- net led_pin: track 0.00 -> 10.4 mm, vias 0 -> 1
- net Net-(D5-A): track 0.00 -> 6.07 mm
- net Temp_SDA: track 24.6 -> 30.4 mm
- net +3.3V: track 127.4 -> 129.9 mm

Commit message: Entrega PRJ4
Parts:
- moved J5 0.55 mm to (94.5, 107.3)
Routing:
- net touch_cs: track 49.4 -> 52.5 mm
- net touch_mosi: track 34.9 -> 32.7 mm
- net oxi_scl: track 33.1 -> 31.0 mm
- net +3.3V: track 129.9 -> 132.0 mm
- net displ_led: track 45.7 -> 47.3 mm
- net displ_mosi: track 36.2 -> 35.1 mm
- net displ_sck: track 37.7 -> 36.8 mm
- net GND: track 0.93 -> 0.00 mm, vias 7 -> 3
- net displ_cs: track 35.8 -> 36.8 mm
- net displ_dc: track 50.6 -> 51.2 mm
